File: PCB/leanometer.brd (EAGLE design)
At the start: 33.3 x 90.4 mm, 45 parts, among them U3 ATMEGA328P_TQFP

Commit message: Changed to 3.3Volt power/logic
Communication between MCU and MPU was stoppping due to difference between logic levels, and highly noisy environment of motorcycle.
Change to all 3.3Volt makes the system much more resilient.
Parts:
- R1, R10, R11, R12, R13, R14, R2, R3, R4, R5, R6, R7, R8, R9: value 470 -> 100
- V_REG: value REG1117-5.0 -> REG1117-3.3
- XTAL: value 16MHz -> 8MHz
Connections:
- net 5V_A renamed 3.3V_A
- net 5V_B renamed 3.3V_B
- net 5V_C renamed 3.3V_C
Changed lines of the file:
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@@
 <attribute name="NAME" x="16.764" y="56.134" size="0.508" layer="26" font="vector" ratio="11" rot="MR0"/>
 </element>
-<element name="R1" library="SparkFun-Resistors" library_urn="urn:adsk.eagle:library:532" package="0805" package3d_urn="urn:adsk.eagle:package:39651/1" value="470" x="7.62" y="87.757" smashed="yes" rot="R90">
+<element name="R1" library="SparkFun-Resistors" library_urn="urn:adsk.eagle:library:532" package="0805" package3d_urn="urn:adsk.eagle:package:39651/1" value="100" x="7.62" y="87.757" smashed="yes" rot="R90">
 <attribute name="PROD_ID" value=" " x="69.85" y="118.237" size="1.778" layer="27" rot="R90" display="off"/>
 </element>
-<element name="R10" library="SparkFun-Resistors" library_urn="urn:adsk.eagle:library:532" package="0805" package3d_urn="urn:adsk.eagle:package:39651/1" value="470" x="21.59" y="77.597" smashed="yes" rot="R270">
+<element name="R10" library="SparkFun-Resistors" library_urn="urn:adsk.eagle:library:532" package="0805" package3d_urn="urn:adsk.eagle:package:39651/1" value="100" x="21.59" y="77.597" smashed="yes" rot="R270">
 <attribute name="PROD_ID" value=" " x="-40.64" y="12.827" size="1.778" layer="27" rot="R270" display="off"/>
 </element>
-<element name="R11" library="SparkFun-Resistors" library_urn="urn:adsk.eagle:library:532" package="0805" package3d_urn="urn:adsk.eagle:package:39651/1" value="470" x="16.51" y="77.597" smashed="yes" rot="R270">
+<element name="R11" library="SparkFun-Resistors" library_urn="urn:adsk.eagle:library:532" package="0805" package3d_urn="urn:adsk.eagle:package:39651/1" value="100" x="16.51" y="77.597" smashed="yes" rot="R270">
 <attribute name="PROD_ID" value=" " x="-49.53" y="62.357" size="1.778" layer="27" rot="R270" display="off"/>
 </element>
-<element name="R12" library="SparkFun-Resistors" library_urn="urn:adsk.eagle:library:532" package="0805" package3d_urn="urn:adsk.eagle:package:39651/1" value="470" x="13.97" y="77.597" smashed="yes" rot="R270">
+<element name="R12" library="SparkFun-Resistors" library_urn="urn:adsk.eagle:library:532" package="0805" package3d_urn="urn:adsk.eagle:package:39651/1" value="100" x="13.97" y="77.597" smashed="yes" rot="R270">
 <attribute name="PROD_ID" value=" " x="-52.07" y="58.547" size="1.778" layer="27" rot="R270" display="off"/>
 </element>
-<element name="R13" library="SparkFun-Resistors" library_urn="urn:adsk.eagle:library:532" package="0805" package3d_urn="urn:adsk.eagle:package:39651/1" value="470" x="16.51" y="87.757" smashed="yes" rot="R90">
+<element name="R13" library="SparkFun-Resistors" library_urn="urn:adsk.eagle:library:532" package="0805" package3d_urn="urn:adsk.eagle:package:39651/1" value="100" x="16.51" y="87.757" smashed="yes" rot="R90">
 <attribute name="PROD_ID" value=" " x="82.55" y="110.617" size="1.778" layer="27" rot="R90" display="off"/>
 </element>
-<element name="R14" library="SparkFun-Resistors" library_urn="urn:adsk.eagle:library:532" package="0805" package3d_urn="urn:adsk.eagle:package:39651/1" value="470" x="13.97" y="87.757" smashed="yes" rot="R90">
+<element name="R14" library="SparkFun-Resistors" library_urn="urn:adsk.eagle:library:532" package="0805" package3d_urn="urn:adsk.eagle:package:39651/1" value="100" x="13.97" y="87.757" smashed="yes" rot="R90">
 <attribute name="PROD_ID" value=" " x="80.01" y="114.427" size="1.778" layer="27" rot="R90" display="off"/>
 </element>
-<element name="R2" library="SparkFun-Resistors" library_urn="urn:adsk.eagle:library:532" package="0805" package3d_urn="urn:adsk.eagle:package:39651/1" value="470" x="10.16" y="87.757" smashed="yes" rot="R90">
+<element name="R2" library="SparkFun-Resistors" library_urn="urn:adsk.eagle:library:532" package="0805" package3d_urn="urn:adsk.eagle:package:39651/1" value="100" x="10.16" y="87.757" smashed="yes" rot="R90">
 <attribute name="PROD_ID" value=" " x="72.39" y="122.047" size="1.778" layer="27" rot="R90" display="off"/>
 </element>
-<element name="R3" library="SparkFun-Resistors" library_urn="urn:adsk.eagle:library:532" package="0805" package3d_urn="urn:adsk.eagle:package:39651/1" value="470" x="7.62" y="77.597" smashed="yes" rot="R270">
+<element name="R3" library="SparkFun-Resistors" library_urn="urn:adsk.eagle:library:532" package="0805" package3d_urn="urn:adsk.eagle:package:39651/1" value="100" x="7.62" y="77.597" smashed="yes" rot="R270">
 <attribute name="PROD_ID" value=" " x="-54.61" y="39.497" size="1.778" layer="27" rot="R270" display="off"/>
 </element>
-<element name="R4" library="SparkFun-Resistors" library_urn="urn:adsk.eagle:library:532" package="0805" package3d_urn="urn:adsk.eagle:package:39651/1" value="470" x="2.54" y="77.597" smashed="yes" rot="R270">
+<element name="R4" library="SparkFun-Resistors" library_urn="urn:adsk.eagle:library:532" package="0805" package3d_urn="urn:adsk.eagle:package:39651/1" value="100" x="2.54" y="77.597" smashed="yes" rot="R270">
 <attribute name="PROD_ID" value=" " x="-59.69" y="35.687" size="1.778" layer="27" rot="R270" display="off"/>
 </element>
-<element name="R5" library="SparkFun-Resistors" library_urn="urn:adsk.eagle:library:532" package="0805" package3d_urn="urn:adsk.eagle:package:39651/1" value="470" x="0" y="77.597" smashed="yes" rot="R270">
+<element name="R5" library="SparkFun-Resistors" library_urn="urn:adsk.eagle:library:532" package="0805" package3d_urn="urn:adsk.eagle:package:39651/1" value="100" x="0" y="77.597" smashed="yes" rot="R270">
 <attribute name="PROD_ID" value=" " x="-62.23" y="31.877" size="1.778" layer="27" rot="R270" display="off"/>
 </element>
-<element name="R6" library="SparkFun-Resistors" library_urn="urn:adsk.eagle:library:532" package="0805" package3d_urn="urn:adsk.eagle:package:39651/1" value="470" x="2.54" y="87.757" smashed="yes" rot="R90">
+<element name="R6" library="SparkFun-Resistors" library_urn="urn:adsk.eagle:library:532" package="0805" package3d_urn="urn:adsk.eagle:package:39651/1" value="100" x="2.54" y="87.757" smashed="yes" rot="R90">
 <attribute name="PROD_ID" value=" " x="64.77" y="137.287" size="1.778" layer="27" rot="R90" display="off"/>
 </element>
-<element name="R7" library="SparkFun-Resistors" library_urn="urn:adsk.eagle:library:532" package="0805" package3d_urn="urn:adsk.eagle:package:39651/1" value="470" x="0" y="87.757" smashed="yes" rot="R90">
+<element name="R7" library="SparkFun-Resistors" library_urn="urn:adsk.eagle:library:532" package="0805" package3d_urn="urn:adsk.eagle:package:39651/1" value="100" x="0" y="87.757" smashed="yes" rot="R90">
 <attribute name="PROD_ID" value=" " x="62.23" y="141.097" size="1.778" layer="27" rot="R90" display="off"/>
 </element>
-<element name="R8" library="SparkFun-Resistors" library_urn="urn:adsk.eagle:library:532" package="0805" package3d_urn="urn:adsk.eagle:package:39651/1" value="470" x="21.59" y="87.757" smashed="yes" rot="R90">
+<element name="R8" library="SparkFun-Resistors" library_urn="urn:adsk.eagle:library:532" package="0805" package3d_urn="urn:adsk.eagle:package:39651/1" value="100" x="21.59" y="87.757" smashed="yes" rot="R90">
 <attribute name="PROD_ID" value=" " x="83.82" y="144.907" size="1.778" layer="27" rot="R90" display="off"/>
 </element>
-<element name="R9" library="SparkFun-Resistors" library_urn="urn:adsk.eagle:library:532" package="0805" package3d_urn="urn:adsk.eagle:package:39651/1" value="470" x="24.13" y="87.757" smashed="yes" rot="R90">
+<element name="R9" library="SparkFun-Resistors" library_urn="urn:adsk.eagle:library:532" package="0805" package3d_urn="urn:adsk.eagle:package:39651/1" value="100" x="24.13" y="87.757" smashed="yes" rot="R90">
 <attribute name="PROD_ID" value=" " x="86.36" y="148.717" size="1.778" layer="27" rot="R90" display="off"/>
 </element>
@@
 <attribute name="VALUE" x="20.574" y="25.7302" size="0.6096" layer="28" font="vector" ratio="20" rot="MR270"/>
 </element>
-<element name="V_REG" library="burr-brown" library_urn="urn:adsk.eagle:library:111" package="SOT223" package3d_urn="urn:adsk.eagle:package:4940/1" value="REG1117-5.0" x="9.906" y="57.531" smashed="yes" rot="MR270">
+<element name="V_REG" library="burr-brown" library_urn="urn:adsk.eagle:library:111" package="SOT223" package3d_urn="urn:adsk.eagle:package:4940/1" value="REG1117-3.3" x="9.906" y="57.531" smashed="yes" rot="MR270">
 <attribute name="MF" value="" x="40.386" y="35.941" size="1.778" layer="28" rot="MR270" display="off"/>
 <attribute name="MPN" value="REG1117" x="40.386" y="35.941" size="1.778" layer="28" rot="MR270" display="off"/>
@@
 <attribute name="VALUE" x="13.208" y="60.833" size="0.762" layer="28" ratio="10" rot="MR0"/>
 </element>
-<element name="XTAL" library="SparkFun-Clocks" library_urn="urn:adsk.eagle:library:511" package="HC49US" package3d_urn="urn:adsk.eagle:package:37515/1" value="16MHz" x="10.033" y="16.764" smashed="yes" rot="MR180">
+<element name="XTAL" library="SparkFun-Clocks" library_urn="urn:adsk.eagle:library:511" package="HC49US" package3d_urn="urn:adsk.eagle:package:37515/1" value="8MHz" x="10.033" y="16.764" smashed="yes" rot="MR180">
 <attribute name="NAME" x="10.033" y="14.224" size="0.6096" layer="26" font="vector" ratio="20" rot="MR180" align="bottom-center"/>
 <attribute name="PROD_ID" value="XTAL-08181" x="60.833" y="57.404" size="1.778" layer="28" rot="MR180" display="off"/>
@@
 <wire x1="1.524" y1="73.152" x2="2.921" y2="71.755" width="0.3048" layer="16"/>
 </signal>
-<signal name="5V_C">
+<signal name="3.3V_C">
 <contactref element="CON_C" pad="1"/>
 <contactref element="LDR" pad="1"/>
@@
 </polygon>
 </signal>
-<signal name="5V_B">
+<signal name="3.3V_B">
 <contactref element="OUT_C1" pad="1"/>
 <contactref element="V_REG" pad="2"/>
@@
 </polygon>
 </signal>
-<signal name="5V_A">
+<signal name="3.3V_A">
 <contactref element="CON_A" pad="3"/>
 <contactref element="MPU" pad="4"/>
